File: hardware/usb2serial-pic14f1454.brd (EAGLE design)
At the start: 46.4 x 28 mm, 14 parts, among them IC1 PIC16F1454, IC2 LP2950-33, J1 USB-SHIELD-A-H, J2 J2

Commit message: Cleanup
Parts:
- C2: value 10uF -> 100nF; device rcl:E2-4 -> rcl:C050-025X075
- moved C2 1.91 mm to (9.53, 16.5), turned to 90 degrees
Connections:
- net +3V3: no longer C2.+
- net GND: now also C2.2; no longer C2.-
- net N$6: now also C2.1
Routing:
- net N$6: track 11.2 -> 17.3 mm
- net +3V3: track 45.9 -> 40.8 mm
Changed lines of the file:
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@@
 <setting verticaltext="up"/>
 </settings>
-<grid distance="0.025" unitdist="inch" unit="mm" style="lines" multiple="1" display="yes" altdistance="0.005" altunitdist="inch" altunit="inch"/>
+<grid distance="0.025" unitdist="inch" unit="mil" style="lines" multiple="1" display="yes" altdistance="0.005" altunitdist="inch" altunit="inch"/>
 <layers>
 <layer number="1" name="Top" color="4" fill="1" visible="yes" active="yes"/>
@@
 <layer number="14" name="Route14" color="1" fill="6" visible="no" active="no"/>
 <layer number="15" name="Route15" color="4" fill="6" visible="no" active="no"/>
-<layer number="16" name="Bottom" color="1" fill="1" visible="yes" active="yes"/>
+<layer number="16" name="Bottom" color="1" fill="1" visible="no" active="yes"/>
 <layer number="17" name="Pads" color="2" fill="1" visible="yes" active="yes"/>
 <layer number="18" name="Vias" color="2" fill="1" visible="yes" active="yes"/>
@@
 <attribute name="VALUE" x="31.2166" y="-0.0254" size="1.27" layer="27" ratio="10" rot="R270"/>
 </element>
-<element name="C2" library="rcl" package="E2-4" value="10uF" x="9.398" y="14.605" smashed="yes" rot="R180">
-<attribute name="NAME" x="6.858" y="15.875" size="1.27" layer="25" font="vector" ratio="10" rot="R90"/>
-<attribute name="VALUE" x="7.239" y="16.764" size="1.27" layer="27" ratio="10" rot="R180"/>
-</element>
 <element name="C3" library="rcl" package="C050-025X075" value="100nF" x="15.24" y="16.51" smashed="yes" rot="R90">
-<attribute name="NAME" x="13.081" y="17.526" size="1.27" layer="25" font="vector" ratio="10" rot="R90"/>
+<attribute name="NAME" x="13.335" y="15.367" size="1.27" layer="25" font="vector" ratio="10" rot="R90"/>
 <attribute name="VALUE" x="18.034" y="13.081" size="1.27" layer="27" ratio="10" rot="R90"/>
 </element>
@@
 <attribute name="NAME" x="38.227" y="17.78" size="1.27" layer="25" ratio="10" rot="R270"/>
 <attribute name="VALUE" x="38.1" y="11.1506" size="1.27" layer="27" ratio="10" rot="R270"/>
+</element>
+<element name="C2" library="rcl" package="C050-025X075" value="100nF" x="9.525" y="16.51" smashed="yes" rot="R90">
+<attribute name="NAME" x="7.62" y="15.367" size="1.27" layer="25" font="vector" ratio="10" rot="R90"/>
+<attribute name="VALUE" x="12.319" y="13.081" size="1.27" layer="27" ratio="10" rot="R90"/>
 </element>
 </elements>
@@
 <contactref element="R1" pad="2"/>
 <contactref element="R3" pad="1"/>
-<contactref element="C2" pad="-"/>
 <contactref element="C3" pad="2"/>
 <contactref element="C1" pad="-"/>
 <contactref element="IC2" pad="GND"/>
 <contactref element="R2" pad="2"/>
+<contactref element="C2" pad="2"/>
 </signal>
 <signal name="N$1">
@@
 </signal>
 <signal name="+3V3">
-<contactref element="C2" pad="+"/>
 <contactref element="C3" pad="1"/>
 <contactref element="IC1" pad="11"/>
 <contactref element="J2" pad="4"/>
-<wire x1="10.414" y1="14.605" x2="14.605" y2="14.605" width="0.3048" layer="16"/>
-<wire x1="14.605" y1="14.605" x2="15.24" y2="13.97" width="0.3048" layer="16"/>
 <wire x1="15.24" y1="13.97" x2="15.24" y2="9.525" width="0.3048" layer="16"/>
 <wire x1="22.86" y1="13.97" x2="27.305" y2="13.97" width="0.3048" layer="16"/>
@@
 <wire x1="8.382" y1="2.54" x2="8.382" y2="4.5" width="0.3048" layer="16"/>
 <wire x1="8.382" y1="4.5" x2="8.382" y2="6.477" width="0.3048" layer="16"/>
-<wire x1="8.382" y1="6.477" x2="10.16" y2="8.255" width="0.3048" layer="16"/>
-<wire x1="10.16" y1="8.255" x2="11.43" y2="8.255" width="0.3048" layer="16"/>
+<contactref element="C2" pad="1"/>
+<wire x1="9.525" y1="13.97" x2="9.525" y2="8.255" width="0.254" layer="16"/>
+<wire x1="9.525" y1="8.255" x2="8.382" y2="7.112" width="0.254" layer="16"/>
+<wire x1="8.382" y1="6.477" x2="8.382" y2="7.112" width="0.254" layer="16"/>
+<wire x1="11.43" y1="8.255" x2="9.525" y2="8.255" width="0.254" layer="16"/>
 </signal>
 <signal name="N$5">
